Commit message: Reverse rotation direction for 11, 15, 21, 25, 31, 35, 41, 45 joints to support legacy joint trajectories.

File: urdf/sweetie_bot_proto2_description.urdf (robot description, URDF)
Before this commit: robot sweetie_bot_proto2_description, 38 links, 37 joints
Joints:
- joint joint11: axis 1 0 0 -> -1 0 0
- joint joint15: axis 1 0 0 -> -1 0 0
- joint joint21: axis 1 0 0 -> -1 0 0
- joint joint25: axis 1 0 0 -> -1 0 0
- joint joint31: axis 1 0 0 -> -1 0 0
- joint joint35: axis 1 0 0 -> -1 0 0
- joint joint41: axis 1 0 0 -> -1 0 0
- joint joint45: axis 1 0 0 -> -1 0 0

File: urdf/sweetie_bot_proto2_description_stl.urdf (robot description, URDF)
Before this commit: robot sweetie_bot_proto2_description, 38 links, 37 joints
Joints:
- joint joint15: axis 1 0 0 -> -1 0 0
- joint joint21: axis 1 0 0 -> -1 0 0
- joint joint25: axis 1 0 0 -> -1 0 0
- joint joint31: axis 1 0 0 -> -1 0 0
- joint joint35: axis 1 0 0 -> -1 0 0
- joint joint41: axis 1 0 0 -> -1 0 0
- joint joint45: axis 1 0 0 -> -1 0 0

Commit message: Set max effort value to DRS-0201 stall torque.

File: urdf/sweetie_bot_proto2_description.urdf (robot description, URDF)
Before this commit: robot sweetie_bot_proto2_description, 38 links, 37 joints
Joints:
- joint joint11: limit lower=-1.5708 upper=1.5708 effort=1000 velocity=0.25 -> lower=-1.5708 upper=1.5708 effort=2.4 velocity=0.25
- joint joint12: limit lower=-1.5708 upper=1.5708 effort=1000 velocity=0.25 -> lower=-1.5708 upper=1.5708 effort=2.4 velocity=0.25
- joint joint13: limit lower=-1.9 upper=1.9 effort=1000 velocity=0.25 -> lower=-1.9 upper=1.9 effort=2.4 velocity=0.25
- joint joint14: limit lower=-1.5708 upper=1.5708 effort=1000 velocity=0.25 -> lower=-1.5708 upper=1.5708 effort=2.4 velocity=0.25
- joint joint15: limit lower=-1.5708 upper=1.5708 effort=1000 velocity=0.25 -> lower=-1.5708 upper=1.5708 effort=2.4 velocity=0.25
- joint joint16: limit lower=-1.5708 upper=1.5708 effort=1000 velocity=0.25 -> lower=-1.5708 upper=1.5708 effort=2.4 velocity=0.25
- joint joint21: limit lower=-1.5708 upper=1.5708 effort=1000 velocity=0.25 -> lower=-1.5708 upper=1.5708 effort=2.4 velocity=0.25
- joint joint22: limit lower=-1.5708 upper=1.5708 effort=1000 velocity=0.25 -> lower=-1.5708 upper=1.5708 effort=2.4 velocity=0.25
- joint joint23: limit lower=-1.9 upper=1.9 effort=1000 velocity=0.25 -> lower=-1.9 upper=1.9 effort=2.4 velocity=0.25
- joint joint24: limit lower=-1.5708 upper=1.5708 effort=1000 velocity=0.25 -> lower=-1.5708 upper=1.5708 effort=2.4 velocity=0.25
- joint joint25: limit lower=-1.5708 upper=1.5708 effort=1000 velocity=0.25 -> lower=-1.5708 upper=1.5708 effort=2.4 velocity=0.25
- joint joint26: limit lower=-1.5708 upper=1.5708 effort=1000 velocity=0.25 -> lower=-1.5708 upper=1.5708 effort=2.4 velocity=0.25
- joint joint31: limit lower=-1.5708 upper=1.5708 effort=1000 velocity=0.25 -> lower=-1.5708 upper=1.5708 effort=2.4 velocity=0.25
- joint joint32: limit lower=-1.5708 upper=1.5708 effort=1000 velocity=0.25 -> lower=-1.5708 upper=1.5708 effort=2.4 velocity=0.25
- joint joint33: limit lower=-1.9 upper=1.9 effort=1000 velocity=0.25 -> lower=-1.9 upper=1.9 effort=2.4 velocity=0.25
- joint joint34: limit lower=-1.5708 upper=1.5708 effort=1000 velocity=0.25 -> lower=-1.5708 upper=1.5708 effort=2.4 velocity=0.25
- joint joint35: limit lower=-1.5708 upper=1.5708 effort=1000 velocity=0.25 -> lower=-1.5708 upper=1.5708 effort=2.4 velocity=0.25
- joint joint36: limit lower=-1.5708 upper=1.5708 effort=1000 velocity=0.25 -> lower=-1.5708 upper=1.5708 effort=2.4 velocity=0.25
- joint joint41: limit lower=-1.5708 upper=1.5708 effort=1000 velocity=0.25 -> lower=-1.5708 upper=1.5708 effort=2.4 velocity=0.25
- joint joint42: limit lower=-1.5708 upper=1.5708 effort=1000 velocity=0.25 -> lower=-1.5708 upper=1.5708 effort=2.4 velocity=0.25
- joint joint43: limit lower=-1.9 upper=1.9 effort=1000 velocity=0.25 -> lower=-1.9 upper=1.9 effort=2.4 velocity=0.25
- joint joint44: limit lower=-1.5708 upper=1.5708 effort=1000 velocity=0.25 -> lower=-1.5708 upper=1.5708 effort=2.4 velocity=0.25
- joint joint45: limit lower=-1.5708 upper=1.5708 effort=1000 velocity=0.25 -> lower=-1.5708 upper=1.5708 effort=2.4 velocity=0.25
- joint joint46: limit lower=-1.5708 upper=1.5708 effort=1000 velocity=0.25 -> lower=-1.5708 upper=1.5708 effort=2.4 velocity=0.25
- joint joint51: limit lower=-1.5708 upper=0.26 effort=1000 velocity=0.25 -> lower=-1.5708 upper=0.26 effort=2.4 velocity=0.25
- joint joint52: limit lower=-1.5708 upper=1.5708 effort=1000 velocity=0.25 -> lower=-1.5708 upper=1.5708 effort=2.4 velocity=0.25
- joint joint53: limit lower=-0.55 upper=1.0 effort=1000 velocity=0.25 -> lower=-0.55 upper=1.0 effort=2.4 velocity=0.25
- joint joint54: limit lower=-1.5708 upper=1.5708 effort=1000 velocity=0.25 -> lower=-1.5708 upper=1.5708 effort=2.4 velocity=0.25
- joint joint55: limit lower=-1.5708 upper=1.5708 effort=1000 velocity=0.25 -> lower=-1.5708 upper=1.5708 effort=2.4 velocity=0.25
- joint joint56: limit lower=-1.5708 upper=1.5708 effort=1000 velocity=0.25 -> lower=-1.5708 upper=1.5708 effort=2.4 velocity=0.25
- joint joint_eyes_focus_x: limit lower=-0.5 upper=0.5 effort=1000 velocity=0.25 -> lower=-0.5 upper=0.5 effort=2.4 velocity=0.25
- joint joint_eyes_focus_y: limit lower=-0.5 upper=0.5 effort=1000 velocity=0.25 -> lower=-0.5 upper=0.5 effort=2.4 velocity=0.25
- joint joint_eyes_focus_z: limit lower=-0.5 upper=0.5 effort=1000 velocity=0.25 -> lower=-0.5 upper=0.5 effort=2.4 velocity=0.25

File: urdf/sweetie_bot_proto2_description_stl.urdf (robot description, URDF)
Before this commit: robot sweetie_bot_proto2_description, 38 links, 37 joints
Joints:
- joint joint11: limit lower=-1.5708 upper=1.5708 effort=1000 velocity=0.25 -> lower=-1.5708 upper=1.5708 effort=2.4 velocity=0.25
- joint joint12: limit lower=-1.5708 upper=1.5708 effort=1000 velocity=0.25 -> lower=-1.5708 upper=1.5708 effort=2.4 velocity=0.25
- joint joint13: limit lower=-1.9 upper=1.9 effort=1000 velocity=0.25 -> lower=-1.9 upper=1.9 effort=2.4 velocity=0.25
- joint joint14: limit lower=-1.5708 upper=1.5708 effort=1000 velocity=0.25 -> lower=-1.5708 upper=1.5708 effort=2.4 velocity=0.25
- joint joint15: limit lower=-1.5708 upper=1.5708 effort=1000 velocity=0.25 -> lower=-1.5708 upper=1.5708 effort=2.4 velocity=0.25
- joint joint16: limit lower=-1.5708 upper=1.5708 effort=1000 velocity=0.25 -> lower=-1.5708 upper=1.5708 effort=2.4 velocity=0.25
- joint joint21: limit lower=-1.5708 upper=1.5708 effort=1000 velocity=0.25 -> lower=-1.5708 upper=1.5708 effort=2.4 velocity=0.25
- joint joint22: limit lower=-1.5708 upper=1.5708 effort=1000 velocity=0.25 -> lower=-1.5708 upper=1.5708 effort=2.4 velocity=0.25
- joint joint23: limit lower=-1.9 upper=1.9 effort=1000 velocity=0.25 -> lower=-1.9 upper=1.9 effort=2.4 velocity=0.25
- joint joint24: limit lower=-1.5708 upper=1.5708 effort=1000 velocity=0.25 -> lower=-1.5708 upper=1.5708 effort=2.4 velocity=0.25
- joint joint25: limit lower=-1.5708 upper=1.5708 effort=1000 velocity=0.25 -> lower=-1.5708 upper=1.5708 effort=2.4 velocity=0.25
- joint joint26: limit lower=-1.5708 upper=1.5708 effort=1000 velocity=0.25 -> lower=-1.5708 upper=1.5708 effort=2.4 velocity=0.25
- joint joint31: limit lower=-1.5708 upper=1.5708 effort=1000 velocity=0.25 -> lower=-1.5708 upper=1.5708 effort=2.4 velocity=0.25
- joint joint32: limit lower=-1.5708 upper=1.5708 effort=1000 velocity=0.25 -> lower=-1.5708 upper=1.5708 effort=2.4 velocity=0.25
- joint joint33: limit lower=-1.9 upper=1.9 effort=1000 velocity=0.25 -> lower=-1.9 upper=1.9 effort=2.4 velocity=0.25
- joint joint34: limit lower=-1.5708 upper=1.5708 effort=1000 velocity=0.25 -> lower=-1.5708 upper=1.5708 effort=2.4 velocity=0.25
- joint joint35: limit lower=-1.5708 upper=1.5708 effort=1000 velocity=0.25 -> lower=-1.5708 upper=1.5708 effort=2.4 velocity=0.25
- joint joint36: limit lower=-1.5708 upper=1.5708 effort=1000 velocity=0.25 -> lower=-1.5708 upper=1.5708 effort=2.4 velocity=0.25
- joint joint41: limit lower=-1.5708 upper=1.5708 effort=1000 velocity=0.25 -> lower=-1.5708 upper=1.5708 effort=2.4 velocity=0.25
- joint joint42: limit lower=-1.5708 upper=1.5708 effort=1000 velocity=0.25 -> lower=-1.5708 upper=1.5708 effort=2.4 velocity=0.25
- joint joint43: limit lower=-1.9 upper=1.9 effort=1000 velocity=0.25 -> lower=-1.9 upper=1.9 effort=2.4 velocity=0.25
- joint joint44: limit lower=-1.5708 upper=1.5708 effort=1000 velocity=0.25 -> lower=-1.5708 upper=1.5708 effort=2.4 velocity=0.25
- joint joint45: limit lower=-1.5708 upper=1.5708 effort=1000 velocity=0.25 -> lower=-1.5708 upper=1.5708 effort=2.4 velocity=0.25
- joint joint46: limit lower=-1.5708 upper=1.5708 effort=1000 velocity=0.25 -> lower=-1.5708 upper=1.5708 effort=2.4 velocity=0.25
- joint joint51: limit lower=-1.5708 upper=0.26 effort=1000 velocity=0.25 -> lower=-1.5708 upper=0.26 effort=2.4 velocity=0.25
- joint joint52: limit lower=-1.5708 upper=1.5708 effort=1000 velocity=0.25 -> lower=-1.5708 upper=1.5708 effort=2.4 velocity=0.25
- joint joint53: limit lower=-0.55 upper=1.0 effort=1000 velocity=0.25 -> lower=-0.55 upper=1.0 effort=2.4 velocity=0.25
- joint joint54: limit lower=-1.5708 upper=1.5708 effort=1000 velocity=0.25 -> lower=-1.5708 upper=1.5708 effort=2.4 velocity=0.25
- joint joint55: limit lower=-1.5708 upper=1.5708 effort=1000 velocity=0.25 -> lower=-1.5708 upper=1.5708 effort=2.4 velocity=0.25
- joint joint56: limit lower=-1.5708 upper=1.5708 effort=1000 velocity=0.25 -> lower=-1.5708 upper=1.5708 effort=2.4 velocity=0.25
- joint joint_eyes_focus_x: limit lower=-0.5 upper=0.5 effort=1000 velocity=0.25 -> lower=-0.5 upper=0.5 effort=2.4 velocity=0.25
- joint joint_eyes_focus_y: limit lower=-0.5 upper=0.5 effort=1000 velocity=0.25 -> lower=-0.5 upper=0.5 effort=2.4 velocity=0.25
- joint joint_eyes_focus_z: limit lower=-0.5 upper=0.5 effort=1000 velocity=0.25 -> lower=-0.5 upper=0.5 effort=2.4 velocity=0.25

Commit message: Rename eyes chain (joint55,joint56->eye_pitch,eye_yaw) add head virtual joints (joint55, joint56).

File: urdf/sweetie_bot_proto2_description.urdf (robot description, URDF)
Before this commit: robot sweetie_bot_proto2_description, 38 links, 37 joints
Links:
- added link eyes_link_pitch
- added link eyes_link_yaw; visual mesh filename=package://sweetie_bot_proto2_description/meshes/arrow.STL
- link bone56: geometry 
Joints:
- added joint eyes_pitch: type revolute, parent bone54, child eyes_link_pitch, origin xyz=0 0 0 rpy=-1.3878E-14 -6.9398E-15 -7.6286E-17, axis 0 -1 0, limit lower=-1.5708 upper=1.5708 effort=2.4 velocity=0.25
- added joint eyes_yaw: type revolute, parent eyes_link_pitch, child eyes_link_yaw, origin xyz=0 0 0 rpy=-1.3878E-14 -6.9398E-15 -7.6286E-17, axis 0 0 -1, limit lower=-1.5708 upper=1.5708 effort=2.4 velocity=0.25
- joint joint55: axis 0 -1 0 -> 0 0 1; origin xyz=0 0 0 rpy=-1.3878E-14 -6.9398E-15 -7.6286E-17 -> xyz=0.12 0.0 -0.02 rpy=0 0 0
- joint joint56: axis 0 0 -1 -> 0 1 0; origin xyz=0 0 0 rpy=-1.3878E-14 -6.9398E-15 -7.6286E-17 -> xyz=0 0 0 rpy=0 0 0

File: urdf/sweetie_bot_proto2_description_stl.urdf (robot description, URDF)
Before this commit: robot sweetie_bot_proto2_description, 38 links, 37 joints
Links:
- added link eyes_link_pitch
- added link eyes_link_yaw; visual mesh filename=package://sweetie_bot_proto2_description/meshes/arrow.STL
- link bone56: geometry 
Joints:
- added joint eyes_pitch: type revolute, parent bone54, child eyes_link_pitch, origin xyz=0 0 0 rpy=-1.3878E-14 -6.9398E-15 -7.6286E-17, axis 0 -1 0, limit lower=-1.5708 upper=1.5708 effort=2.4 velocity=0.25
- added joint eyes_yaw: type revolute, parent eyes_link_pitch, child eyes_link_yaw, origin xyz=0 0 0 rpy=-1.3878E-14 -6.9398E-15 -7.6286E-17, axis 0 0 -1, limit lower=-1.5708 upper=1.5708 effort=2.4 velocity=0.25
- joint joint55: axis 0 -1 0 -> 0 0 1; origin xyz=0 0 0 rpy=-1.3878E-14 -6.9398E-15 -7.6286E-17 -> xyz=0.12 0.0 -0.02 rpy=0 0 0
- joint joint56: axis 0 0 -1 -> 0 1 0; origin xyz=0 0 0 rpy=-1.3878E-14 -6.9398E-15 -7.6286E-17 -> xyz=0 0 0 rpy=0 0 0

Commit message: joint54 limits fixed

File: urdf/sweetie_bot_proto2_description.urdf (robot description, URDF)
Before this commit: robot sweetie_bot_proto2_description, 40 links, 39 joints
Joints:
- joint joint54: limit lower=-1.5708 upper=1.5708 effort=2.4 velocity=0.25 -> lower=-0.4 upper=0.4 effort=2.4 velocity=0.25

File: urdf/sweetie_bot_proto2_description_dynamics.urdf (robot description, URDF)
Before this commit: robot sweetie_bot_proto2_description, 27 links, 26 joints
Joints:
- joint joint54: limit lower=-1.5708 upper=1.5708 effort=2.4 velocity=0.25 -> lower=-0.4 upper=0.4 effort=2.4 velocity=0.25

File: urdf/sweetie_bot_proto2_description_stl.urdf (robot description, URDF)
Before this commit: robot sweetie_bot_proto2_description, 40 links, 39 joints
Joints:
- joint joint54: limit lower=-1.5708 upper=1.5708 effort=2.4 velocity=0.25 -> lower=-0.4 upper=0.4 effort=2.4 velocity=0.25
