Commit message: Change effort and velocity default limits.

File: urdf/sweetie_bot_proto2_description.urdf (robot description, URDF)
Before this commit: robot sweetie_bot_proto2_description, 40 links, 39 joints
Joints:
- joint eyes_pitch: limit lower=-1.5708 upper=1.5708 effort=2.4 velocity=0.25 -> lower=-1.5708 upper=1.5708 effort=0.24 velocity=6.2832
- joint eyes_yaw: limit lower=-1.5708 upper=1.5708 effort=2.4 velocity=0.25 -> lower=-1.5708 upper=1.5708 effort=0.24 velocity=6.2832
- joint joint11: limit lower=-1.5708 upper=1.5708 effort=2.4 velocity=0.25 -> lower=-1.5708 upper=1.5708 effort=0.24 velocity=1.5708
- joint joint12: limit lower=-1.5708 upper=1.5708 effort=2.4 velocity=0.25 -> lower=-1.5708 upper=1.5708 effort=0.24 velocity=1.5708
- joint joint13: limit lower=-1.9 upper=1.9 effort=2.4 velocity=0.25 -> lower=-1.9 upper=1.9 effort=0.24 velocity=1.5708
- joint joint14: limit lower=-1.5708 upper=1.5708 effort=2.4 velocity=0.25 -> lower=-1.5708 upper=1.5708 effort=0.24 velocity=1.5708
- joint joint15: limit lower=-1.5708 upper=1.5708 effort=2.4 velocity=0.25 -> lower=-1.5708 upper=1.5708 effort=0.24 velocity=1.5708
- joint joint16: limit lower=-1.5708 upper=1.5708 effort=2.4 velocity=0.25 -> lower=-1.5708 upper=1.5708 effort=0.24 velocity=6.2832
- joint joint21: limit lower=-1.5708 upper=1.5708 effort=2.4 velocity=0.25 -> lower=-1.5708 upper=1.5708 effort=0.24 velocity=1.5708
- joint joint22: limit lower=-1.5708 upper=1.5708 effort=2.4 velocity=0.25 -> lower=-1.5708 upper=1.5708 effort=0.24 velocity=1.5708
- joint joint23: limit lower=-1.9 upper=1.9 effort=2.4 velocity=0.25 -> lower=-1.9 upper=1.9 effort=0.24 velocity=1.5708
- joint joint24: limit lower=-1.5708 upper=1.5708 effort=2.4 velocity=0.25 -> lower=-1.5708 upper=1.5708 effort=0.24 velocity=1.5708
- joint joint25: limit lower=-1.5708 upper=1.5708 effort=2.4 velocity=0.25 -> lower=-1.5708 upper=1.5708 effort=0.24 velocity=1.5708
- joint joint26: limit lower=-1.5708 upper=1.5708 effort=2.4 velocity=0.25 -> lower=-1.5708 upper=1.5708 effort=0.24 velocity=6.2832
- joint joint31: limit lower=-1.5708 upper=1.5708 effort=2.4 velocity=0.25 -> lower=-1.5708 upper=1.5708 effort=0.24 velocity=1.5708
- joint joint32: limit lower=-1.5708 upper=1.5708 effort=2.4 velocity=0.25 -> lower=-1.5708 upper=1.5708 effort=0.24 velocity=1.5708
- joint joint33: limit lower=-1.9 upper=1.9 effort=2.4 velocity=0.25 -> lower=-1.9 upper=1.9 effort=0.24 velocity=1.5708
- joint joint34: limit lower=-1.5708 upper=1.5708 effort=2.4 velocity=0.25 -> lower=-1.5708 upper=1.5708 effort=0.24 velocity=1.5708
- joint joint35: limit lower=-1.5708 upper=1.5708 effort=2.4 velocity=0.25 -> lower=-1.5708 upper=1.5708 effort=0.24 velocity=1.5708
- joint joint36: limit lower=-1.5708 upper=1.5708 effort=2.4 velocity=0.25 -> lower=-1.5708 upper=1.5708 effort=0.24 velocity=6.2832
- joint joint41: limit lower=-1.5708 upper=1.5708 effort=2.4 velocity=0.25 -> lower=-1.5708 upper=1.5708 effort=0.24 velocity=1.5708
- joint joint42: limit lower=-1.5708 upper=1.5708 effort=2.4 velocity=0.25 -> lower=-1.5708 upper=1.5708 effort=0.24 velocity=1.5708
- joint joint43: limit lower=-1.9 upper=1.9 effort=2.4 velocity=0.25 -> lower=-1.9 upper=1.9 effort=0.24 velocity=1.5708
- joint joint44: limit lower=-1.5708 upper=1.5708 effort=2.4 velocity=0.25 -> lower=-1.5708 upper=1.5708 effort=0.24 velocity=1.5708
- joint joint45: limit lower=-1.5708 upper=1.5708 effort=2.4 velocity=0.25 -> lower=-1.5708 upper=1.5708 effort=0.24 velocity=1.5708
- joint joint46: limit lower=-1.5708 upper=1.5708 effort=2.4 velocity=0.25 -> lower=-1.5708 upper=1.5708 effort=0.24 velocity=6.2832
- joint joint51: limit lower=-1.5708 upper=0.26 effort=2.4 velocity=0.25 -> lower=-1.5708 upper=0.26 effort=0.24 velocity=1.5708
- joint joint52: limit lower=-1.5708 upper=1.5708 effort=2.4 velocity=0.25 -> lower=-1.5708 upper=1.5708 effort=0.24 velocity=1.5708
- joint joint53: limit lower=-0.55 upper=1.0 effort=2.4 velocity=0.25 -> lower=-0.55 upper=1.0 effort=0.24 velocity=1.5708
- joint joint54: limit lower=-0.4 upper=0.4 effort=2.4 velocity=0.25 -> lower=-0.4 upper=0.4 effort=0.24 velocity=1.5708
- joint joint55: limit lower=-1.5708 upper=1.5708 effort=2.4 velocity=0.25 -> lower=-1.5708 upper=1.5708 effort=0.24 velocity=6.2832
- joint joint56: limit lower=-1.5708 upper=1.5708 effort=2.4 velocity=0.25 -> lower=-1.5708 upper=1.5708 effort=0.24 velocity=6.2832
- joint joint_eyes_focus_x: limit lower=-0.5 upper=0.5 effort=2.4 velocity=0.25 -> lower=-0.5 upper=0.5 effort=0.24 velocity=1.5708
- joint joint_eyes_focus_y: limit lower=-0.5 upper=0.5 effort=2.4 velocity=0.25 -> lower=-0.5 upper=0.5 effort=0.24 velocity=1.5708
- joint joint_eyes_focus_z: limit lower=-0.5 upper=0.5 effort=2.4 velocity=0.25 -> lower=-0.5 upper=0.5 effort=0.24 velocity=1.5708

File: urdf/sweetie_bot_proto2_description_dynamics.urdf (robot description, URDF)
Before this commit: robot sweetie_bot_proto2_description, 27 links, 26 joints
Joints:
- joint joint11: limit lower=-1.5708 upper=1.5708 effort=2.4 velocity=0.25 -> lower=-1.5708 upper=1.5708 effort=0.24 velocity=1.5708
- joint joint12: limit lower=-1.5708 upper=1.5708 effort=2.4 velocity=0.25 -> lower=-1.5708 upper=1.5708 effort=0.24 velocity=1.5708
- joint joint13: limit lower=-1.9 upper=1.9 effort=2.4 velocity=0.25 -> lower=-1.9 upper=1.9 effort=0.24 velocity=1.5708
- joint joint14: limit lower=-1.5708 upper=1.5708 effort=2.4 velocity=0.25 -> lower=-1.5708 upper=1.5708 effort=0.24 velocity=1.5708
- joint joint15: limit lower=-1.5708 upper=1.5708 effort=2.4 velocity=0.25 -> lower=-1.5708 upper=1.5708 effort=0.24 velocity=1.5708
- joint joint21: limit lower=-1.5708 upper=1.5708 effort=2.4 velocity=0.25 -> lower=-1.5708 upper=1.5708 effort=0.24 velocity=1.5708
- joint joint22: limit lower=-1.5708 upper=1.5708 effort=2.4 velocity=0.25 -> lower=-1.5708 upper=1.5708 effort=0.24 velocity=1.5708
- joint joint23: limit lower=-1.9 upper=1.9 effort=2.4 velocity=0.25 -> lower=-1.9 upper=1.9 effort=0.24 velocity=1.5708
- joint joint24: limit lower=-1.5708 upper=1.5708 effort=2.4 velocity=0.25 -> lower=-1.5708 upper=1.5708 effort=0.24 velocity=1.5708
- joint joint25: limit lower=-1.5708 upper=1.5708 effort=2.4 velocity=0.25 -> lower=-1.5708 upper=1.5708 effort=0.24 velocity=1.5708
- joint joint31: limit lower=-1.5708 upper=1.5708 effort=2.4 velocity=0.25 -> lower=-1.5708 upper=1.5708 effort=0.24 velocity=1.5708
- joint joint32: limit lower=-1.5708 upper=1.5708 effort=2.4 velocity=0.25 -> lower=-1.5708 upper=1.5708 effort=0.24 velocity=1.5708
- joint joint33: limit lower=-1.9 upper=1.9 effort=2.4 velocity=0.25 -> lower=-1.9 upper=1.9 effort=0.24 velocity=1.5708
- joint joint34: limit lower=-1.5708 upper=1.5708 effort=2.4 velocity=0.25 -> lower=-1.5708 upper=1.5708 effort=0.24 velocity=1.5708
- joint joint35: limit lower=-1.5708 upper=1.5708 effort=2.4 velocity=0.25 -> lower=-1.5708 upper=1.5708 effort=0.24 velocity=1.5708
- joint joint41: limit lower=-1.5708 upper=1.5708 effort=2.4 velocity=0.25 -> lower=-1.5708 upper=1.5708 effort=0.24 velocity=1.5708
- joint joint42: limit lower=-1.5708 upper=1.5708 effort=2.4 velocity=0.25 -> lower=-1.5708 upper=1.5708 effort=0.24 velocity=1.5708
- joint joint43: limit lower=-1.9 upper=1.9 effort=2.4 velocity=0.25 -> lower=-1.9 upper=1.9 effort=0.24 velocity=1.5708
- joint joint44: limit lower=-1.5708 upper=1.5708 effort=2.4 velocity=0.25 -> lower=-1.5708 upper=1.5708 effort=0.24 velocity=1.5708
- joint joint45: limit lower=-1.5708 upper=1.5708 effort=2.4 velocity=0.25 -> lower=-1.5708 upper=1.5708 effort=0.24 velocity=1.5708
- joint joint51: limit lower=-1.5708 upper=0.26 effort=2.4 velocity=0.25 -> lower=-1.5708 upper=0.26 effort=0.24 velocity=1.5708
- joint joint52: limit lower=-1.5708 upper=1.5708 effort=2.4 velocity=0.25 -> lower=-1.5708 upper=1.5708 effort=0.24 velocity=1.5708
- joint joint53: limit lower=-0.55 upper=1.0 effort=2.4 velocity=0.25 -> lower=-0.55 upper=1.0 effort=0.24 velocity=1.5708
- joint joint54: limit lower=-0.4 upper=0.4 effort=2.4 velocity=0.25 -> lower=-0.4 upper=0.4 effort=0.24 velocity=1.5708

File: urdf/sweetie_bot_proto2_description_stl.urdf (robot description, URDF)
Before this commit: robot sweetie_bot_proto2_description, 40 links, 39 joints
Joints:
- joint eyes_pitch: limit lower=-1.5708 upper=1.5708 effort=2.4 velocity=0.25 -> lower=-1.5708 upper=1.5708 effort=0.24 velocity=1.5708
- joint eyes_yaw: limit lower=-1.5708 upper=1.5708 effort=2.4 velocity=0.25 -> lower=-1.5708 upper=1.5708 effort=0.24 velocity=1.5708
- joint joint11: limit lower=-1.5708 upper=1.5708 effort=2.4 velocity=0.25 -> lower=-1.5708 upper=1.5708 effort=0.24 velocity=1.5708
- joint joint12: limit lower=-1.5708 upper=1.5708 effort=2.4 velocity=0.25 -> lower=-1.5708 upper=1.5708 effort=0.24 velocity=1.5708
- joint joint13: limit lower=-1.9 upper=1.9 effort=2.4 velocity=0.25 -> lower=-1.9 upper=1.9 effort=0.24 velocity=1.5708
- joint joint14: limit lower=-1.5708 upper=1.5708 effort=2.4 velocity=0.25 -> lower=-1.5708 upper=1.5708 effort=0.24 velocity=1.5708
- joint joint15: limit lower=-1.5708 upper=1.5708 effort=2.4 velocity=0.25 -> lower=-1.5708 upper=1.5708 effort=0.24 velocity=1.5708
- joint joint16: limit lower=-1.5708 upper=1.5708 effort=2.4 velocity=0.25 -> lower=-1.5708 upper=1.5708 effort=0.24 velocity=6.2832
- joint joint21: limit lower=-1.5708 upper=1.5708 effort=2.4 velocity=0.25 -> lower=-1.5708 upper=1.5708 effort=0.24 velocity=1.5708
- joint joint22: limit lower=-1.5708 upper=1.5708 effort=2.4 velocity=0.25 -> lower=-1.5708 upper=1.5708 effort=0.24 velocity=1.5708
- joint joint23: limit lower=-1.9 upper=1.9 effort=2.4 velocity=0.25 -> lower=-1.9 upper=1.9 effort=0.24 velocity=1.5708
- joint joint24: limit lower=-1.5708 upper=1.5708 effort=2.4 velocity=0.25 -> lower=-1.5708 upper=1.5708 effort=0.24 velocity=1.5708
- joint joint25: limit lower=-1.5708 upper=1.5708 effort=2.4 velocity=0.25 -> lower=-1.5708 upper=1.5708 effort=0.24 velocity=1.5708
- joint joint26: limit lower=-1.5708 upper=1.5708 effort=2.4 velocity=0.25 -> lower=-1.5708 upper=1.5708 effort=0.24 velocity=6.2832
- joint joint31: limit lower=-1.5708 upper=1.5708 effort=2.4 velocity=0.25 -> lower=-1.5708 upper=1.5708 effort=0.24 velocity=1.5708
- joint joint32: limit lower=-1.5708 upper=1.5708 effort=2.4 velocity=0.25 -> lower=-1.5708 upper=1.5708 effort=0.24 velocity=1.5708
- joint joint33: limit lower=-1.9 upper=1.9 effort=2.4 velocity=0.25 -> lower=-1.9 upper=1.9 effort=0.24 velocity=1.5708
- joint joint34: limit lower=-1.5708 upper=1.5708 effort=2.4 velocity=0.25 -> lower=-1.5708 upper=1.5708 effort=0.24 velocity=1.5708
- joint joint35: limit lower=-1.5708 upper=1.5708 effort=2.4 velocity=0.25 -> lower=-1.5708 upper=1.5708 effort=0.24 velocity=1.5708
- joint joint36: limit lower=-1.5708 upper=1.5708 effort=2.4 velocity=0.25 -> lower=-1.5708 upper=1.5708 effort=0.24 velocity=6.2832
- joint joint41: limit lower=-1.5708 upper=1.5708 effort=2.4 velocity=0.25 -> lower=-1.5708 upper=1.5708 effort=0.24 velocity=1.5708
- joint joint42: limit lower=-1.5708 upper=1.5708 effort=2.4 velocity=0.25 -> lower=-1.5708 upper=1.5708 effort=0.24 velocity=1.5708
- joint joint43: limit lower=-1.9 upper=1.9 effort=2.4 velocity=0.25 -> lower=-1.9 upper=1.9 effort=0.24 velocity=1.5708
- joint joint44: limit lower=-1.5708 upper=1.5708 effort=2.4 velocity=0.25 -> lower=-1.5708 upper=1.5708 effort=0.24 velocity=1.5708
- joint joint45: limit lower=-1.5708 upper=1.5708 effort=2.4 velocity=0.25 -> lower=-1.5708 upper=1.5708 effort=0.24 velocity=1.5708
- joint joint46: limit lower=-1.5708 upper=1.5708 effort=2.4 velocity=0.25 -> lower=-1.5708 upper=1.5708 effort=0.24 velocity=6.2832
- joint joint51: limit lower=-1.5708 upper=0.26 effort=2.4 velocity=0.25 -> lower=-1.5708 upper=0.26 effort=0.24 velocity=1.5708
- joint joint52: limit lower=-1.5708 upper=1.5708 effort=2.4 velocity=0.25 -> lower=-1.5708 upper=1.5708 effort=0.24 velocity=1.5708
- joint joint53: limit lower=-0.55 upper=1.0 effort=2.4 velocity=0.25 -> lower=-0.55 upper=1.0 effort=0.24 velocity=1.5708
- joint joint54: limit lower=-0.4 upper=0.4 effort=2.4 velocity=0.25 -> lower=-0.4 upper=0.4 effort=0.24 velocity=1.5708
- joint joint55: limit lower=-1.5708 upper=1.5708 effort=2.4 velocity=0.25 -> lower=-1.5708 upper=1.5708 effort=0.24 velocity=6.2832
- joint joint56: limit lower=-1.5708 upper=1.5708 effort=2.4 velocity=0.25 -> lower=-1.5708 upper=1.5708 effort=0.24 velocity=6.2832
- joint joint_eyes_focus_x: limit lower=-0.5 upper=0.5 effort=2.4 velocity=0.25 -> lower=-0.5 upper=0.5 effort=0.24 velocity=1.5708
- joint joint_eyes_focus_y: limit lower=-0.5 upper=0.5 effort=2.4 velocity=0.25 -> lower=-0.5 upper=0.5 effort=0.24 velocity=1.5708
- joint joint_eyes_focus_z: limit lower=-0.5 upper=0.5 effort=2.4 velocity=0.25 -> lower=-0.5 upper=0.5 effort=0.24 velocity=1.5708

Commit message: Fix KDL message about base_link inertia: move inertia in fictive link attached to base_link.

File: urdf/sweetie_bot_proto2_description.urdf (robot description, URDF)
Before this commit: robot sweetie_bot_proto2_description, 40 links, 39 joints
Links:
- added link base_link_inertia, mass 0.455451435671981
- link base_link: mass 0.455451435671981 -> None
Joints:
- added joint fictive_base_joint: type fixed, parent base_link, child base_link_inertia

File: urdf/sweetie_bot_proto2_description_stl.urdf (robot description, URDF)
Before this commit: robot sweetie_bot_proto2_description, 40 links, 39 joints
Links:
- added link base_link_inertia, mass 0.455451435671981
- link base_link: mass 0.455451435671981 -> None
Joints:
- added joint fictive_base_joint: type fixed, parent base_link, child base_link_inertia

Commit message: Introduce hoof1..hoof4 frames. Probably temporary, until gait generator is unable to use contact model to calculalte contact points.

File: urdf/sweetie_bot_proto2_description.urdf (robot description, URDF)
Before this commit: robot sweetie_bot_proto2_description, 41 links, 40 joints
Links:
- added link hoof1
- added link hoof2
- added link hoof3
- added link hoof4
Joints:
- added joint joint_hoof1: type fixed, parent bone15, child hoof1, origin xyz=0 0 -0.03 rpy=0 0 0
- added joint joint_hoof2: type fixed, parent bone25, child hoof2, origin xyz=0 0 -0.03 rpy=0 0 0
- added joint joint_hoof3: type fixed, parent bone35, child hoof3, origin xyz=0 0 -0.03 rpy=0 0 0
- added joint joint_hoof4: type fixed, parent bone45, child hoof4, origin xyz=0 0 -0.03 rpy=0 0 0
