Commit message: Updated dynamic robot model

File: urdf/sweetie_bot_proto2_description.urdf (robot description, URDF)
Before this commit: robot sweetie_bot_proto2_description, 45 links, 44 joints
Links:
- link base_link_inertia: mass 0.455451435671981 -> 0.971931208405
- link bone11: mass 0.0926240684197254 -> 0.105587079651
- link bone12: mass 0.0180633663571699 -> 0.0185022042823
- link bone13: mass 0.0573118289119351 -> 0.0651096345569
- link bone14: mass 0.0926240684197256 -> 0.105587079787
- link bone15: mass 0.0231901119311412 -> 0.0234095309231
- link bone21: mass 0.0926240685372407 -> 0.105587079651
- link bone22: mass 0.0180633663571699 -> 0.0185022042823
- link bone23: mass 0.0573118289119352 -> 0.0651096347113
- link bone24: mass 0.0926240686547557 -> 0.105587079787
- link bone25: mass 0.0231901117609318 -> 0.0234095313367
- link bone31: mass 0.0926240684197254 -> 0.105587079515
- link bone32: mass 0.01806336635717 -> 0.0185022042823
- link bone33: mass 0.0573118289119353 -> 0.0651096345569
- link bone34: mass 0.0926240686547557 -> 0.105587079787
- link bone35: mass 0.0231901117341147 -> 0.0234095310833
- link bone41: mass 0.0926240684197254 -> 0.105587079742
- link bone42: mass 0.01806336635717 -> 0.0185022042823
- link bone43: mass 0.0573118289904725 -> 0.0651096346928
- link bone44: mass 0.0926240684982629 -> 0.105587079805
- link bone45: mass 0.023190112165723 -> 0.0234095308805
- link bone51: mass 0.0896127849103651 -> 0.102575796082
- link bone52: mass 0.00518639804635041 -> 0.00540581700891
- link bone53: mass 0.0480856556054743 -> 0.0556640423453
- link bone54: mass 0.208663345422344 -> 0.230098004362
- link eye_left: mass 0.0352933751936015 -> None; geometry 
- link eye_right: mass 0.0352933751936015 -> None; geometry 
- link screen_left: mass None -> 0.034287324936; geometry collision mesh filename=package://sweetie_bot_proto2_description/meshes/screen_left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; visual mesh filename=package://sweetie_bot_proto2_description/meshes/screen_left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
- link screen_right: mass None -> 0.034287324936; geometry collision mesh filename=package://sweetie_bot_proto2_description/meshes/screen_righ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; visual mesh filename=package://sweetie_bot_proto2_description/meshes/screen_righ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
Joints:
- joint eye_left: axis 0 0 0 -> 0.0 0.0 0.0; origin xyz=0.070269 0.033627 0.0060879 rpy=0 0 0 -> xyz=0.0700895479365 0.0337909018151 0.00614838727403 rpy=-3.44033294541e-16 3.15829803493e-14 2.50910403565e-14
- joint eye_right: axis 0 0 0 -> 0.0 0.0 0.0; origin xyz=0.070268 -0.033628 0.0060848 rpy=0 0 0 -> xyz=0.0700889457663 -0.0337914070959 0.00614523448994 rpy=-3.69982123334e-16 3.16973967665e-14 2.50355292053e-14
- joint eyes_pitch: axis 0 -1 0 -> 0.0 -1.0 0.0; origin xyz=0 0 0 rpy=-1.3878E-14 -6.9398E-15 -7.6286E-17 -> xyz=0.0 0.0 0.0 rpy=-1.3878e-14 -6.9398e-15 -7.6286e-17
- joint eyes_yaw: axis 0 0 -1 -> 0.0 0.0 -1.0; origin xyz=0 0 0 rpy=-1.3878E-14 -6.9398E-15 -7.6286E-17 -> xyz=0.0 0.0 0.0 rpy=-1.3878e-14 -6.9398e-15 -7.6286e-17
- joint joint11: axis -1 0 0 -> -1.0 0.0 0.0; origin xyz=0.080425 0.037 -0.0275 rpy=-6.123E-17 0 0 -> xyz=0.080425 0.037 -0.0275 rpy=3.7797374822e-14 -3.4914813431e-15 -4.81230658754e-15
- joint joint12: axis 0 -1 0 -> 0.0 -1.0 0.0; origin xyz=0 0 0 rpy=-3.4694E-15 0 0 -> xyz=0.0 0.0 0.0 rpy=0.0 -3.54776255454e-31 0.0
- joint joint13: axis 0 -1 0 -> 0.0 -1.0 0.0; origin xyz=0 0 -0.08 rpy=-6.9389E-16 0 0 -> xyz=0.0 0.0 -0.08 rpy=-3.16413562018e-15 3.4914813431e-15 4.81230658754e-15
- joint joint14: axis 0 -1 0 -> 0.0 -1.0 0.0; origin xyz=0 0.0016 -0.09605 rpy=4.1633E-15 0 0 -> xyz=0.0 0.0016 -0.09605 rpy=-3.88578058619e-16 6.93889390398e-18 2.17881268583e-15
- joint joint15: axis -1 0 0 -> -1.0 0.0 0.0; origin xyz=0 0 0 rpy=1.1102E-14 0 0 -> xyz=0.0 0.0 0.0 rpy=0.0 -1.12103877146e-44 0.0
- joint joint16: axis 0 0 1 -> 0.0 0.0 1.0; origin xyz=0 0 0 rpy=0 0 0 -> xyz=0.0 0.0 0.0 rpy=0.0 0.0 0.0
- joint joint21: axis -1 0 0 -> -1.0 0.0 0.0; origin xyz=0.080425 -0.037 -0.0275 rpy=-6.123E-17 0 0 -> xyz=0.080425 -0.037 -0.0275 rpy=3.54699451234e-15 4.38428390321e-16 -1.54361546163e-14
- joint joint22: axis 0 -1 0 -> 0.0 -1.0 0.0; origin xyz=0 0 0 rpy=-1.0408E-14 0 0 -> xyz=0.0 0.0 0.0 rpy=0.0 1.6185064457e-32 0.0
- joint joint23: axis 0 -1 0 -> 0.0 -1.0 0.0; origin xyz=0 0 -0.08 rpy=6.245E-15 0 0 -> xyz=0.0 0.0 -0.08 rpy=-7.77156117238e-15 -4.38428390321e-16 1.54361546163e-14
- joint joint24: axis 0 -1 0 -> 0.0 -1.0 0.0; origin xyz=0 -0.0016 -0.09605 rpy=4.1633E-15 0 0 -> xyz=0.0 -0.0016 -0.09605 rpy=-6.38378239159e-15 4.4408920985e-16 -7.77156117238e-16
- joint joint25: axis -1 0 0 -> -1.0 0.0 0.0; origin xyz=0 0 0 rpy=-2.7756E-15 0 0 -> xyz=0.0 0.0 0.0 rpy=0.0 1.23259516441e-32 0.0
- joint joint26: axis 0 0 1 -> 0.0 0.0 1.0; origin xyz=0 0 0 rpy=0 0 0 -> xyz=0.0 0.0 0.0 rpy=0.0 0.0 0.0
- joint joint31: axis -1 0 0 -> -1.0 0.0 0.0; origin xyz=-0.080425 0.037 -0.0275 rpy=-6.123E-17 0 0 -> xyz=-0.080425 0.037 -0.0275 rpy=-3.54455505745e-15 -9.51716093093e-30 -6.52476541856e-14
- joint joint32: axis 0 -1 0 -> 0.0 -1.0 0.0; origin xyz=0 0 0 rpy=3.4694E-15 0 0 -> xyz=0.0 0.0 0.0 rpy=0.0 0.0 0.0
- joint joint33: axis 0 -1 0 -> 0.0 -1.0 0.0; origin xyz=0 0 -0.08 rpy=-7.6328E-15 0 0 -> xyz=0.0 0.0 -0.08 rpy=-6.80011602583e-16 -2.217567417e-28 6.52476541856e-14
- joint joint34: axis 0 -1 0 -> 0.0 -1.0 0.0; origin xyz=0 0.0016 -0.09605 rpy=4.1633E-15 0 0 -> xyz=0.0 0.0016 -0.09605 rpy=7.88258347484e-15 -9.15933995316e-15 2.39154391688e-17
- joint joint35: axis -1 0 0 -> -1.0 0.0 0.0; origin xyz=0 0 0 rpy=-1.6653E-14 0 0 -> xyz=0.0 0.0 0.0 rpy=0.0 8.89474285511e-32 0.0
- joint joint36: axis 0 0 1 -> 0.0 0.0 1.0; origin xyz=0 0 0 rpy=0 0 0 -> xyz=0.0 0.0 0.0 rpy=0.0 0.0 0.0
- joint joint41: axis -1 0 0 -> -1.0 0.0 0.0; origin xyz=-0.080425 -0.037 -0.0275 rpy=-6.123E-17 0 0 -> xyz=-0.080425 -0.037 -0.0275 rpy=-3.64169957211e-15 -5.31264912662e-17 -3.51471262493e-14
- joint joint42: axis 0 -1 0 -> 0.0 -1.0 0.0; origin xyz=0 0 0 rpy=-3.1225E-15 0 0 -> xyz=0.0 0.0 0.0 rpy=0.0 1.40160664338e-33 0.0
- joint joint43: axis 0 -1 0 -> 0.0 -1.0 0.0; origin xyz=0 0 -0.08 rpy=7.2858E-15 0 0 -> xyz=0.0 0.0 -0.08 rpy=7.74380559676e-15 5.31264912661e-17 3.51471262493e-14
- joint joint44: axis 0 -1 0 -> 0.0 -1.0 0.0; origin xyz=0 -0.0016 -0.09605 rpy=-4.1633E-15 0 0 -> xyz=0.0 -0.0016 -0.09605 rpy=-1.42386102908e-14 -8.88910258347e-17 -2.32357620616e-14
- joint joint45: axis -1 0 0 -> -1.0 0.0 0.0; origin xyz=0 0 0 rpy=2.7756E-15 0 0 -> xyz=0.0 0.0 0.0 rpy=0.0 -1.31403502749e-34 0.0
- joint joint46: axis 0 0 1 -> 0.0 0.0 1.0; origin xyz=0 0 0 rpy=0 0 0 -> xyz=0.0 0.0 0.0 rpy=0.0 0.0 0.0
- joint joint51: axis 0 -1 0 -> 0.0 -1.0 0.0; origin xyz=0.088 0 0.0235 rpy=-6.5958E-16 -2.803E-13 1.7163E-29 -> xyz=0.088 0.0 0.0235 rpy=-4.57151135523e-15 0.0 0.0
- joint joint52: axis 0 0 1 -> 0.0 0.0 1.0; origin xyz=0 -0.00315 0.06705 rpy=-2.2859E-16 2.8041E-13 1.6778E-28 -> xyz=0.0 -0.00314999999999 0.06705 rpy=-3.30198557404e-15 -6.86083134749e-15 3.72722466096e-14
- joint joint53: axis 0 -1 0 -> 0.0 -1.0 0.0; origin xyz=0 0 0 rpy=-4.792E-17 -1.817E-16 -1.5026E-31 -> xyz=0.0 0.0 0.0 rpy=-5.14406073106e-16 6.86083134749e-15 -3.72722466096e-14
- joint joint54: axis 1 0 0 -> 1.0 0.0 0.0; origin xyz=0 0.00315 0.0246 rpy=-1.6564E-27 3.835E-14 3.3551E-29 -> xyz=0.0 0.00314999999999 0.0246 rpy=2.77555756156e-14 0.0 0.0
- joint joint55: axis 0 0 1 -> 0.0 0.0 1.0; origin xyz=0.12 0.0 -0.02 rpy=0 0 0 -> xyz=0.12 0.0 -0.02 rpy=0.0 0.0 0.0
- joint joint56: axis 0 1 0 -> 0.0 1.0 0.0; origin xyz=0 0 0 rpy=0 0 0 -> xyz=0.0 0.0 0.0 rpy=0.0 0.0 0.0
- joint joint_eyes_focus_x: axis 1 0 0 -> 1.0 0.0 0.0; origin xyz=0 0 0 rpy=0 0 0 -> xyz=0.0 0.0 0.0 rpy=0.0 0.0 0.0
- joint joint_eyes_focus_y: axis 0 1 0 -> 0.0 1.0 0.0; origin xyz=0 0 0 rpy=0 0 0 -> xyz=0.0 0.0 0.0 rpy=0.0 0.0 0.0
- joint joint_eyes_focus_z: axis 0 0 1 -> 0.0 0.0 1.0; origin xyz=0 0 0 rpy=0 0 0 -> xyz=0.0 0.0 0.0 rpy=0.0 0.0 0.0
- joint joint_hoof1: origin xyz=0 0 -0.03 rpy=0 0 0 -> xyz=0.0 0.0 -0.03 rpy=0.0 0.0 0.0
- joint joint_hoof2: origin xyz=0 0 -0.03 rpy=0 0 0 -> xyz=0.0 0.0 -0.03 rpy=0.0 0.0 0.0
- joint joint_hoof3: origin xyz=0 0 -0.03 rpy=0 0 0 -> xyz=0.0 0.0 -0.03 rpy=0.0 0.0 0.0
- joint joint_hoof4: origin xyz=0 0 -0.03 rpy=0 0 0 -> xyz=0.0 0.0 -0.03 rpy=0.0 0.0 0.0
- joint screen_left: axis 0 0 0 -> 0.0 0.0 0.0; origin xyz=0.070269 0.033627 0.0060879 rpy=1.5708 -0.24435 2.4435 -> xyz=0.0700895479365 0.0337909018151 0.00614838727403 rpy=1.5707963268 -0.244346095279 2.44346095279
- joint screen_right: axis 0 0 0 -> 0.0 0.0 0.0; origin xyz=0.070268 -0.033628 0.0060848 rpy=1.5708 0.24435 0.69813 -> xyz=0.0700889457663 -0.0337914070959 0.00614523448994 rpy=1.5707963268 0.244346095279 0.698131700799

File: urdf/sweetie_bot_proto2_description_dynamics.urdf (robot description, URDF)
Before this commit: robot sweetie_bot_proto2_description, 27 links, 26 joints
Links:
- link base_link: mass 0.455451435671981 -> 0.971931208405
- link bone11: mass 0.0926240684197254 -> 0.105587079651
- link bone12: mass 0.0180633663571699 -> 0.0185022042823
- link bone13: mass 0.0573118289119351 -> 0.0651096345569
- link bone14: mass 0.0926240684197256 -> 0.105587079787
- link bone15: mass 0.0231901119311412 -> 0.0234095309231
- link bone21: mass 0.0926240685372407 -> 0.105587079651
- link bone22: mass 0.0180633663571699 -> 0.0185022042823
- link bone23: mass 0.0573118289119352 -> 0.0651096347113
- link bone24: mass 0.0926240686547557 -> 0.105587079787
- link bone25: mass 0.0231901117609318 -> 0.0234095313367
- link bone31: mass 0.0926240684197254 -> 0.105587079515
- link bone32: mass 0.01806336635717 -> 0.0185022042823
- link bone33: mass 0.0573118289119353 -> 0.0651096345569
- link bone34: mass 0.0926240686547557 -> 0.105587079787
- link bone35: mass 0.0231901117341147 -> 0.0234095310833
- link bone41: mass 0.0926240684197254 -> 0.105587079742
- link bone42: mass 0.01806336635717 -> 0.0185022042823
- link bone43: mass 0.0573118289904725 -> 0.0651096346928
- link bone44: mass 0.0926240684982629 -> 0.105587079805
- link bone45: mass 0.023190112165723 -> 0.0234095308805
- link bone51: mass 0.0896127849103651 -> 0.102575796082
- link bone52: mass 0.00518639804635041 -> 0.00540581700891
- link bone53: mass 0.0480856556054743 -> 0.0556640423453
- link bone54: mass 0.208663345422344 -> 0.230098004362
- link eye_left: mass 0.0352933751936015 -> None; geometry 
- link eye_right: mass 0.0352933751936015 -> None; geometry 
Joints:
- joint eye_left: axis 0 0 0 -> 0.0 0.0 0.0; origin xyz=0.070269 0.033627 0.0060879 rpy=0 0 0 -> xyz=0.0700895479365 0.0337909018151 0.00614838727403 rpy=-3.44033294541e-16 3.15829803493e-14 2.50910403565e-14
- joint eye_right: axis 0 0 0 -> 0.0 0.0 0.0; origin xyz=0.070268 -0.033628 0.0060848 rpy=0 0 0 -> xyz=0.0700889457663 -0.0337914070959 0.00614523448994 rpy=-3.69982123334e-16 3.16973967665e-14 2.50355292053e-14
- joint joint11: axis -1 0 0 -> -1.0 0.0 0.0; origin xyz=0.080425 0.037 -0.0275 rpy=-6.123E-17 0 0 -> xyz=0.080425 0.037 -0.0275 rpy=3.7797374822e-14 -3.4914813431e-15 -4.81230658754e-15
- joint joint12: axis 0 -1 0 -> 0.0 -1.0 0.0; origin xyz=0 0 0 rpy=-3.4694E-15 0 0 -> xyz=0.0 0.0 0.0 rpy=0.0 -3.54776255454e-31 0.0
- joint joint13: axis 0 -1 0 -> 0.0 -1.0 0.0; origin xyz=0 0 -0.08 rpy=-6.9389E-16 0 0 -> xyz=0.0 0.0 -0.08 rpy=-3.16413562018e-15 3.4914813431e-15 4.81230658754e-15
- joint joint14: axis 0 -1 0 -> 0.0 -1.0 0.0; origin xyz=0 0.0016 -0.09605 rpy=4.1633E-15 0 0 -> xyz=0.0 0.0016 -0.09605 rpy=-3.88578058619e-16 6.93889390398e-18 2.17881268583e-15
- joint joint15: axis -1 0 0 -> -1.0 0.0 0.0; origin xyz=0 0 0 rpy=1.1102E-14 0 0 -> xyz=0.0 0.0 0.0 rpy=0.0 -1.12103877146e-44 0.0
- joint joint21: axis -1 0 0 -> -1.0 0.0 0.0; origin xyz=0.080425 -0.037 -0.0275 rpy=-6.123E-17 0 0 -> xyz=0.080425 -0.037 -0.0275 rpy=3.54699451234e-15 4.38428390321e-16 -1.54361546163e-14
- joint joint22: axis 0 -1 0 -> 0.0 -1.0 0.0; origin xyz=0 0 0 rpy=-1.0408E-14 0 0 -> xyz=0.0 0.0 0.0 rpy=0.0 1.6185064457e-32 0.0
- joint joint23: axis 0 -1 0 -> 0.0 -1.0 0.0; origin xyz=0 0 -0.08 rpy=6.245E-15 0 0 -> xyz=0.0 0.0 -0.08 rpy=-7.77156117238e-15 -4.38428390321e-16 1.54361546163e-14
- joint joint24: axis 0 -1 0 -> 0.0 -1.0 0.0; origin xyz=0 -0.0016 -0.09605 rpy=4.1633E-15 0 0 -> xyz=0.0 -0.0016 -0.09605 rpy=-6.38378239159e-15 4.4408920985e-16 -7.77156117238e-16
- joint joint25: axis -1 0 0 -> -1.0 0.0 0.0; origin xyz=0 0 0 rpy=-2.7756E-15 0 0 -> xyz=0.0 0.0 0.0 rpy=0.0 1.23259516441e-32 0.0
- joint joint31: axis -1 0 0 -> -1.0 0.0 0.0; origin xyz=-0.080425 0.037 -0.0275 rpy=-6.123E-17 0 0 -> xyz=-0.080425 0.037 -0.0275 rpy=-3.54455505745e-15 -9.51716093093e-30 -6.52476541856e-14
- joint joint32: axis 0 -1 0 -> 0.0 -1.0 0.0; origin xyz=0 0 0 rpy=3.4694E-15 0 0 -> xyz=0.0 0.0 0.0 rpy=0.0 0.0 0.0
- joint joint33: axis 0 -1 0 -> 0.0 -1.0 0.0; origin xyz=0 0 -0.08 rpy=-7.6328E-15 0 0 -> xyz=0.0 0.0 -0.08 rpy=-6.80011602583e-16 -2.217567417e-28 6.52476541856e-14
- joint joint34: axis 0 -1 0 -> 0.0 -1.0 0.0; origin xyz=0 0.0016 -0.09605 rpy=4.1633E-15 0 0 -> xyz=0.0 0.0016 -0.09605 rpy=7.88258347484e-15 -9.15933995316e-15 2.39154391688e-17
- joint joint35: axis -1 0 0 -> -1.0 0.0 0.0; origin xyz=0 0 0 rpy=-1.6653E-14 0 0 -> xyz=0.0 0.0 0.0 rpy=0.0 8.89474285511e-32 0.0
- joint joint41: axis -1 0 0 -> -1.0 0.0 0.0; origin xyz=-0.080425 -0.037 -0.0275 rpy=-6.123E-17 0 0 -> xyz=-0.080425 -0.037 -0.0275 rpy=-3.64169957211e-15 -5.31264912662e-17 -3.51471262493e-14
- joint joint42: axis 0 -1 0 -> 0.0 -1.0 0.0; origin xyz=0 0 0 rpy=-3.1225E-15 0 0 -> xyz=0.0 0.0 0.0 rpy=0.0 1.40160664338e-33 0.0
- joint joint43: axis 0 -1 0 -> 0.0 -1.0 0.0; origin xyz=0 0 -0.08 rpy=7.2858E-15 0 0 -> xyz=0.0 0.0 -0.08 rpy=7.74380559676e-15 5.31264912661e-17 3.51471262493e-14
- joint joint44: axis 0 -1 0 -> 0.0 -1.0 0.0; origin xyz=0 -0.0016 -0.09605 rpy=-4.1633E-15 0 0 -> xyz=0.0 -0.0016 -0.09605 rpy=-1.42386102908e-14 -8.88910258347e-17 -2.32357620616e-14
- joint joint45: axis -1 0 0 -> -1.0 0.0 0.0; origin xyz=0 0 0 rpy=2.7756E-15 0 0 -> xyz=0.0 0.0 0.0 rpy=0.0 -1.31403502749e-34 0.0
- joint joint51: axis 0 -1 0 -> 0.0 -1.0 0.0; origin xyz=0.088 0 0.0235 rpy=-6.5958E-16 -2.803E-13 1.7163E-29 -> xyz=0.088 0.0 0.0235 rpy=-4.57151135523e-15 0.0 0.0
- joint joint52: axis 0 0 1 -> 0.0 0.0 1.0; origin xyz=0 -0.00315 0.06705 rpy=-2.2859E-16 2.8041E-13 1.6778E-28 -> xyz=0.0 -0.00314999999999 0.06705 rpy=-3.30198557404e-15 -6.86083134749e-15 3.72722466096e-14
- joint joint53: axis 0 -1 0 -> 0.0 -1.0 0.0; origin xyz=0 0 0 rpy=-4.792E-17 -1.817E-16 -1.5026E-31 -> xyz=0.0 0.0 0.0 rpy=-5.14406073106e-16 6.86083134749e-15 -3.72722466096e-14
- joint joint54: axis 1 0 0 -> 1.0 0.0 0.0; origin xyz=0 0.00315 0.0246 rpy=-1.6564E-27 3.835E-14 3.3551E-29 -> xyz=0.0 0.00314999999999 0.0246 rpy=2.77555756156e-14 0.0 0.0

Commit message: Alternative hoof construction

File: urdf/sweetie_bot_proto2_description.urdf (robot description, URDF)
Before this commit: robot sweetie_bot_proto2, 45 links, 44 joints
Links:
- link bone15: mass 0.0234095309231 -> 0.0200023100057
- link bone25: mass 0.0234095313367 -> 0.0200023097747
- link bone34: mass 0.105587079787 -> 0.105587079677
- link bone35: mass 0.0234095310833 -> 0.0200023099234
- link bone43: mass 0.0651096346928 -> 0.0651096346478
- link bone45: mass 0.0234095308805 -> 0.0200023102673
- link bone54: mass 0.230098004362 -> 0.230099528944
Joints:
- joint joint34: origin xyz=0.0 0.0016 -0.09605 rpy=7.88258347484e-15 -9.15933995316e-15 2.39154391688e-17 -> xyz=0.0 0.0 -0.09605 rpy=6.93889390391e-15 0.0 0.0
- joint joint35: origin xyz=0.0 0.0 0.0 rpy=0.0 8.89474285511e-32 0.0 -> xyz=0.0 0.0 0.0 rpy=2.22044604925e-14 2.02615701994e-13 -3.14159265359
- joint joint44: origin xyz=0.0 -0.0016 -0.09605 rpy=-1.42386102908e-14 -8.88910258347e-17 -2.32357620616e-14 -> xyz=0.0 0.0 -0.09605 rpy=-1.52655665886e-14 0.0 0.0
- joint joint45: origin xyz=0.0 0.0 0.0 rpy=0.0 -1.31403502749e-34 0.0 -> xyz=0.0 0.0 0.0 rpy=-8.32667268469e-15 -2.72004641033e-13 -3.14159265359

File: urdf/sweetie_bot_proto2_description_dynamics.urdf (robot description, URDF)
Before this commit: robot sweetie_bot_proto2, 27 links, 26 joints
Links:
- link bone15: mass 0.0234095309231 -> 0.0200023100057
- link bone25: mass 0.0234095313367 -> 0.0200023097747
- link bone34: mass 0.105587079787 -> 0.105587079677
- link bone35: mass 0.0234095310833 -> 0.0200023099234
- link bone43: mass 0.0651096346928 -> 0.0651096346478
- link bone45: mass 0.0234095308805 -> 0.0200023102673
- link bone54: mass 0.230098004362 -> 0.230099528944
Joints:
- joint joint34: origin xyz=0.0 0.0016 -0.09605 rpy=7.88258347484e-15 -9.15933995316e-15 2.39154391688e-17 -> xyz=0.0 0.0 -0.09605 rpy=6.93889390391e-15 0.0 0.0
- joint joint35: origin xyz=0.0 0.0 0.0 rpy=0.0 8.89474285511e-32 0.0 -> xyz=0.0 0.0 0.0 rpy=2.22044604925e-14 2.02615701994e-13 -3.14159265359
- joint joint44: origin xyz=0.0 -0.0016 -0.09605 rpy=-1.42386102908e-14 -8.88910258347e-17 -2.32357620616e-14 -> xyz=0.0 0.0 -0.09605 rpy=-1.52655665886e-14 0.0 0.0
- joint joint45: origin xyz=0.0 0.0 0.0 rpy=0.0 -1.31403502749e-34 0.0 -> xyz=0.0 0.0 0.0 rpy=-8.32667268469e-15 -2.72004641033e-13 -3.14159265359

Commit message: Increase limits for joint*4 joints,

File: urdf/sweetie_bot_proto2_description.urdf (robot description, URDF)
Before this commit: robot sweetie_bot_proto2, 45 links, 44 joints
Joints:
- joint joint14: limit lower=-1.5708 upper=1.5708 effort=0.24 velocity=1.5708 -> lower=-1.7 upper=1.7 effort=0.24 velocity=1.5708
- joint joint24: limit lower=-1.5708 upper=1.5708 effort=0.24 velocity=1.5708 -> lower=-1.7 upper=1.7 effort=0.24 velocity=1.5708
- joint joint34: limit lower=-1.5708 upper=1.5708 effort=0.24 velocity=1.5708 -> lower=-1.7 upper=1.7 effort=0.24 velocity=1.5708
- joint joint44: limit lower=-1.5708 upper=1.5708 effort=0.24 velocity=1.5708 -> lower=-1.7 upper=1.7 effort=0.24 velocity=1.5708

File: urdf/sweetie_bot_proto2_description_dynamics.urdf (robot description, URDF)
Before this commit: robot sweetie_bot_proto2, 27 links, 26 joints
Joints:
- joint joint14: limit lower=-1.5708 upper=1.5708 effort=0.24 velocity=1.5708 -> lower=-1.7 upper=1.7 effort=0.24 velocity=1.5708
- joint joint24: limit lower=-1.5708 upper=1.5708 effort=0.24 velocity=1.5708 -> lower=-1.7 upper=1.7 effort=0.24 velocity=1.5708
- joint joint34: limit lower=-1.5708 upper=1.5708 effort=0.24 velocity=1.5708 -> lower=-1.7 upper=1.7 effort=0.24 velocity=1.5708
- joint joint44: limit lower=-1.5708 upper=1.5708 effort=0.24 velocity=1.5708 -> lower=-1.7 upper=1.7 effort=0.24 velocity=1.5708

Commit message: Remove eyes focus joints and links.

File: urdf/sweetie_bot_proto2_description.urdf (robot description, URDF)
Before this commit: robot sweetie_bot_proto2, 45 links, 44 joints
Links:
- removed link link_eyes_x
- removed link link_eyes_y
- removed link link_eyes_z
Joints:
- removed joint joint_eyes_focus_x
- removed joint joint_eyes_focus_y
- removed joint joint_eyes_focus_z
