Commit message: Fix effort limits for joints (0.24 -> 2.4).

File: urdf/sweetie_bot_proto2_description.urdf (robot description, URDF)
Before this commit: robot sweetie_bot_proto2, 42 links, 41 joints
Joints:
- joint eyes_pitch: limit lower=-1.5708 upper=1.5708 effort=0.24 velocity=6.2832 -> lower=-1.5708 upper=1.5708 effort=2.4 velocity=6.2832
- joint eyes_yaw: limit lower=-1.5708 upper=1.5708 effort=0.24 velocity=6.2832 -> lower=-1.5708 upper=1.5708 effort=2.4 velocity=6.2832
- joint joint11: limit lower=-1.5708 upper=1.5708 effort=0.24 velocity=1.5708 -> lower=-1.5708 upper=1.5708 effort=2.4 velocity=1.5708
- joint joint12: limit lower=-1.5708 upper=1.5708 effort=0.24 velocity=1.5708 -> lower=-1.5708 upper=1.5708 effort=2.4 velocity=1.5708
- joint joint13: limit lower=-1.9 upper=1.9 effort=0.24 velocity=1.5708 -> lower=-1.9 upper=1.9 effort=2.4 velocity=1.5708
- joint joint14: limit lower=-1.7 upper=1.7 effort=0.24 velocity=1.5708 -> lower=-1.7 upper=1.7 effort=2.4 velocity=1.5708
- joint joint15: limit lower=-1.5708 upper=1.5708 effort=0.24 velocity=1.5708 -> lower=-1.5708 upper=1.5708 effort=2.4 velocity=1.5708
- joint joint16: limit lower=-1.5708 upper=1.5708 effort=0.24 velocity=6.2832 -> lower=-1.5708 upper=1.5708 effort=2.4 velocity=6.2832
- joint joint21: limit lower=-1.5708 upper=1.5708 effort=0.24 velocity=1.5708 -> lower=-1.5708 upper=1.5708 effort=2.4 velocity=1.5708
- joint joint22: limit lower=-1.5708 upper=1.5708 effort=0.24 velocity=1.5708 -> lower=-1.5708 upper=1.5708 effort=2.4 velocity=1.5708
- joint joint23: limit lower=-1.9 upper=1.9 effort=0.24 velocity=1.5708 -> lower=-1.9 upper=1.9 effort=2.4 velocity=1.5708
- joint joint24: limit lower=-1.7 upper=1.7 effort=0.24 velocity=1.5708 -> lower=-1.7 upper=1.7 effort=2.4 velocity=1.5708
- joint joint25: limit lower=-1.5708 upper=1.5708 effort=0.24 velocity=1.5708 -> lower=-1.5708 upper=1.5708 effort=2.4 velocity=1.5708
- joint joint26: limit lower=-1.5708 upper=1.5708 effort=0.24 velocity=6.2832 -> lower=-1.5708 upper=1.5708 effort=2.4 velocity=6.2832
- joint joint31: limit lower=-1.5708 upper=1.5708 effort=0.24 velocity=1.5708 -> lower=-1.5708 upper=1.5708 effort=2.4 velocity=1.5708
- joint joint32: limit lower=-1.5708 upper=1.5708 effort=0.24 velocity=1.5708 -> lower=-1.5708 upper=1.5708 effort=2.4 velocity=1.5708
- joint joint33: limit lower=-1.9 upper=1.9 effort=0.24 velocity=1.5708 -> lower=-1.9 upper=1.9 effort=2.4 velocity=1.5708
- joint joint34: limit lower=-1.7 upper=1.7 effort=0.24 velocity=1.5708 -> lower=-1.7 upper=1.7 effort=2.4 velocity=1.5708
- joint joint35: limit lower=-1.5708 upper=1.5708 effort=0.24 velocity=1.5708 -> lower=-1.5708 upper=1.5708 effort=2.4 velocity=1.5708
- joint joint36: limit lower=-1.5708 upper=1.5708 effort=0.24 velocity=6.2832 -> lower=-1.5708 upper=1.5708 effort=2.4 velocity=6.2832
- joint joint41: limit lower=-1.5708 upper=1.5708 effort=0.24 velocity=1.5708 -> lower=-1.5708 upper=1.5708 effort=2.4 velocity=1.5708
- joint joint42: limit lower=-1.5708 upper=1.5708 effort=0.24 velocity=1.5708 -> lower=-1.5708 upper=1.5708 effort=2.4 velocity=1.5708
- joint joint43: limit lower=-1.9 upper=1.9 effort=0.24 velocity=1.5708 -> lower=-1.9 upper=1.9 effort=2.4 velocity=1.5708
- joint joint44: limit lower=-1.7 upper=1.7 effort=0.24 velocity=1.5708 -> lower=-1.7 upper=1.7 effort=2.4 velocity=1.5708
- joint joint45: limit lower=-1.5708 upper=1.5708 effort=0.24 velocity=1.5708 -> lower=-1.5708 upper=1.5708 effort=2.4 velocity=1.5708
- joint joint46: limit lower=-1.5708 upper=1.5708 effort=0.24 velocity=6.2832 -> lower=-1.5708 upper=1.5708 effort=2.4 velocity=6.2832
- joint joint51: limit lower=-1.5708 upper=0.26 effort=0.24 velocity=1.5708 -> lower=-1.5708 upper=0.26 effort=2.4 velocity=1.5708
- joint joint52: limit lower=-1.5708 upper=1.5708 effort=0.24 velocity=1.5708 -> lower=-1.5708 upper=1.5708 effort=2.4 velocity=1.5708
- joint joint53: limit lower=-0.55 upper=1.0 effort=0.24 velocity=1.5708 -> lower=-0.55 upper=1.0 effort=2.4 velocity=1.5708
- joint joint54: limit lower=-0.4 upper=0.4 effort=0.24 velocity=1.5708 -> lower=-0.4 upper=0.4 effort=2.4 velocity=1.5708
- joint joint55: limit lower=-1.5708 upper=1.5708 effort=0.24 velocity=6.2832 -> lower=-1.5708 upper=1.5708 effort=2.4 velocity=6.2832
- joint joint56: limit lower=-1.5708 upper=1.5708 effort=0.24 velocity=6.2832 -> lower=-1.5708 upper=1.5708 effort=2.4 velocity=6.2832

File: urdf/sweetie_bot_proto2_description_dynamics.urdf (robot description, URDF)
Before this commit: robot sweetie_bot_proto2, 27 links, 26 joints
Joints:
- joint joint11: limit lower=-1.5708 upper=1.5708 effort=0.24 velocity=1.5708 -> lower=-1.5708 upper=1.5708 effort=2.4 velocity=1.5708

Commit message: Fix eyes pitch and yaw angles semantic.

File: urdf/sweetie_bot_proto2_description.urdf (robot description, URDF)
Before this commit: robot sweetie_bot_proto2, 42 links, 41 joints
Links:
- link eyes_link_pitch: geometry visual mesh filename=package://sweetie_bot_proto2_description/meshes/arrow.STL
- link eyes_link_yaw: geometry 
Joints:
- joint eyes_pitch: parent bone54 -> eyes_link_yaw
- joint eyes_yaw: origin xyz=0.0 0.0 0.0 rpy=-1.3878e-14 -6.9398e-15 -7.6286e-17 -> xyz=0.0 0.0 0.0 rpy=0.0 0.0 0.0; parent eyes_link_pitch -> bone54

Commit message: Add 'camera_link_simulation' frame to connect simulated camera.

File: urdf/sweetie_bot_proto2_description.urdf (robot description, URDF)
Before this commit: robot sweetie_bot_proto2, 42 links, 41 joints
Links:
- added link camera_link
- added link camera_link_simulation
Joints:
- added joint camera_joint: type fixed, parent bone54, child camera_link, origin xyz=0.095 0.0 0.055 rpy=1.5708 0.0 1.5708, axis 0.0 0.0 0.0
- added joint camera_joint_simulation: type fixed, parent base_link, child camera_link_simulation, origin xyz=0.183 0.0 0.11515 rpy=1.5708 0.0 1.5708, axis 0.0 0.0 0.0
